File: nummacro.kicad_pcb (KiCad board)
At the start: 2 copper layers, 348.3 x 121 mm, 367 parts, among them CON1 ISP, J1 USB_B, Q1 Q_NPN_BEC, SW1 SW_RESET, SW2 SW_HWB, U1 AT90USB1286, Y1 16Mhz

Commit message: Rerouted, migrated to standard KiCad keyboard footprints, moved to USB-C to address durability issues. Added holed for PCB-mounted stabilisers for standalone usage.
Parts:
- removed the C4 at (356.8, 121.8)
- removed the C5 at (356.8, 123.7)
- removed the C6 at (356.7, 119.8)
- removed the LED_1 at (39.7, 28.4)
- removed LED_28, LED_35, LED_43, LED_50, LED_64, LED_71, LED_75, LED_76, LED_79, LED_80, LED_85: MX_LED, LED_THT:LED_D3.0mm
- removed the R29 at (152.8, 127.5)
- removed the R44 at (223.7, 54.0)
- removed the R5 at (43.8, 107.6)
- removed the R72 at (361.2, 28.1)
- removed the R83 at (152.8, 62.9)
- removed the R84 at (172.1, 62.9)
- added C2: 100n, Capacitor_SMD:C_0805_2012Metric_Pad1.15x1.40mm_HandSolder, B.Cu at (355.0, 120.2)
- added C3: 100n, Capacitor_SMD:C_0805_2012Metric_Pad1.15x1.40mm_HandSolder, B.Cu at (355.0, 122.1)
- added C7: 100n, Capacitor_SMD:C_0805_2012Metric_Pad1.15x1.40mm_HandSolder, B.Cu at (369.9, 125.3)
- added C8: 10uF, Capacitor_SMD:C_0805_2012Metric_Pad1.15x1.40mm_HandSolder, B.Cu at (369.9, 123.3)
- added D88: MBR130LSFT1G, Diode_SMD:D_PowerDI-123, B.Cu at (373.2, 124.9)
- added G***: LOGO, ingwaz, B.Cu at (123.9, 133.2)
- added LED_5: Led_Small, LED_THT:LED_D3.0mm, F.Cu at (135.1, 52.6)
- added LED_8: Led_Small, LED_THT:LED_D3.0mm, F.Cu at (192.0, 52.7)
- added LED_BKSPC1: Led_Small, LED_THT:LED_D3.0mm, F.Cu at (296.8, 52.2)
- added LED_F10: Led_Small, LED_THT:LED_D3.0mm, F.Cu at (268.1, 29.1)
- added LED_F5: Led_Small, LED_THT:LED_D3.0mm, F.Cu at (162.8, 28.8)
- added LED_F8: Led_Small, LED_THT:LED_D3.0mm, F.Cu at (220.0, 28.9)
- added LED_HOME1: Led_Small, LED_THT:LED_D3.0mm, F.Cu at (349.5, 52.9)
- added LED_INS1: Led_Small, LED_THT:LED_D3.0mm, F.Cu at (330.6, 52.9)
- added LED_PGUP1: Led_Small, LED_THT:LED_D3.0mm, F.Cu at (368.6, 52.9)
- added LED_PRN1: Led_Small, LED_THT:LED_D3.0mm, F.Cu at (330.7, 28.7)
- added LED_SCRL1: Led_Small, LED_THT:LED_D3.0mm, F.Cu at (349.7, 28.7)
- added LED_TILDE1: Led_Small, LED_THT:LED_D3.0mm, F.Cu at (40.0, 52.6)
- added R10: 1K, Resistor_SMD:R_0805_2012Metric_Pad1.15x1.40mm_HandSolder, B.Cu at (350.6, 90.0)
- added R34: 470, Resistor_SMD:R_0805_2012Metric_Pad1.15x1.40mm_HandSolder, B.Cu at (129.3, 52.7)
- added R49: 470, Resistor_SMD:R_0805_2012Metric_Pad1.15x1.40mm_HandSolder, B.Cu at (186.2, 52.8)
- added R87: 470, Resistor_SMD:R_0805_2012Metric_Pad1.15x1.40mm_HandSolder, B.Cu at (343.7, 71.7)
- added R88: 470, Resistor_SMD:R_0805_2012Metric_Pad1.15x1.40mm_HandSolder, B.Cu at (343.5, 110.8)
- added REF**: OSHW-Logo2_14.6x12mm_SilkScreen, Symbol:OSHW-Logo2_14.6x12mm_SilkScreen, B.Cu at (268.5, 110.9)
- D1, D41, D87: footprint Diode_SMD:D_SOD-123 -> Diode_SMD:D_MiniMELF
- D10: renamed from D52; footprint Diode_SMD:D_SOD-123 -> Diode_SMD:D_MiniMELF
- D11: renamed from D2; footprint Diode_SMD:D_SOD-123 -> Diode_SMD:D_MiniMELF
- D12: renamed from D19; footprint Diode_SMD:D_SOD-123 -> Diode_SMD:D_MiniMELF
- D13: renamed from D65; footprint Diode_SMD:D_SOD-123 -> Diode_SMD:D_MiniMELF
- D14: renamed from D36; footprint Diode_SMD:D_SOD-123 -> Diode_SMD:D_MiniMELF
- D15: renamed from D79; footprint Diode_SMD:D_SOD-123 -> Diode_SMD:D_MiniMELF
- D16: renamed from D53; footprint Diode_SMD:D_SOD-123 -> Diode_SMD:D_MiniMELF
- D17: renamed from D3; footprint Diode_SMD:D_SOD-123 -> Diode_SMD:D_MiniMELF
- D18: renamed from D20; footprint Diode_SMD:D_SOD-123 -> Diode_SMD:D_MiniMELF
- D19: renamed from D66; footprint Diode_SMD:D_SOD-123 -> Diode_SMD:D_MiniMELF
- D2: renamed from D17; footprint Diode_SMD:D_SOD-123 -> Diode_SMD:D_MiniMELF
- D20: renamed from D37; footprint Diode_SMD:D_SOD-123 -> Diode_SMD:D_MiniMELF
- D21: renamed from D54; footprint Diode_SMD:D_SOD-123 -> Diode_SMD:D_MiniMELF
- D22: renamed from D4; footprint Diode_SMD:D_SOD-123 -> Diode_SMD:D_MiniMELF
- D23: renamed from D21; footprint Diode_SMD:D_SOD-123 -> Diode_SMD:D_MiniMELF
- D24: renamed from D67; footprint Diode_SMD:D_SOD-123 -> Diode_SMD:D_MiniMELF
- D25: renamed from D38; footprint Diode_SMD:D_SOD-123 -> Diode_SMD:D_MiniMELF
- D26: renamed from D55; footprint Diode_SMD:D_SOD-123 -> Diode_SMD:D_MiniMELF
- D27: renamed from D5; footprint Diode_SMD:D_SOD-123 -> Diode_SMD:D_MiniMELF
- D28: renamed from D22; footprint Diode_SMD:D_SOD-123 -> Diode_SMD:D_MiniMELF
- D29: renamed from D68; footprint Diode_SMD:D_SOD-123 -> Diode_SMD:D_MiniMELF
- D3: renamed from D77; footprint Diode_SMD:D_SOD-123 -> Diode_SMD:D_MiniMELF
- D30: renamed from D39; footprint Diode_SMD:D_SOD-123 -> Diode_SMD:D_MiniMELF
- D31: renamed from D56; footprint Diode_SMD:D_SOD-123 -> Diode_SMD:D_MiniMELF
- D32: renamed from D23; footprint Diode_SMD:D_SOD-123 -> Diode_SMD:D_MiniMELF
- D33: renamed from D69; footprint Diode_SMD:D_SOD-123 -> Diode_SMD:D_MiniMELF
- D34: renamed from D80; footprint Diode_SMD:D_SOD-123 -> Diode_SMD:D_MiniMELF
- D35: renamed from D6; footprint Diode_SMD:D_SOD-123 -> Diode_SMD:D_MiniMELF
- D36: renamed from D40; footprint Diode_SMD:D_SOD-123 -> Diode_SMD:D_MiniMELF
- D37: renamed from D57; footprint Diode_SMD:D_SOD-123 -> Diode_SMD:D_MiniMELF
- D38: renamed from D24; footprint Diode_SMD:D_SOD-123 -> Diode_SMD:D_MiniMELF
- D39: renamed from D70; footprint Diode_SMD:D_SOD-123 -> Diode_SMD:D_MiniMELF
- D4: renamed from D34; footprint Diode_SMD:D_SOD-123 -> Diode_SMD:D_MiniMELF
- D40: renamed from D7; footprint Diode_SMD:D_SOD-123 -> Diode_SMD:D_MiniMELF
- D42: renamed from D58; footprint Diode_SMD:D_SOD-123 -> Diode_SMD:D_MiniMELF
- D43: renamed from D25; footprint Diode_SMD:D_SOD-123 -> Diode_SMD:D_MiniMELF
- D44: renamed from D71; footprint Diode_SMD:D_SOD-123 -> Diode_SMD:D_MiniMELF
- D45: renamed from D8; footprint Diode_SMD:D_SOD-123 -> Diode_SMD:D_MiniMELF
- D46: renamed from D42; footprint Diode_SMD:D_SOD-123 -> Diode_SMD:D_MiniMELF
- D47: renamed from D59; footprint Diode_SMD:D_SOD-123 -> Diode_SMD:D_MiniMELF
- D48: renamed from D26; footprint Diode_SMD:D_SOD-123 -> Diode_SMD:D_MiniMELF
- D49: renamed from D72; footprint Diode_SMD:D_SOD-123 -> Diode_SMD:D_MiniMELF
- D5: renamed from D51; footprint Diode_SMD:D_SOD-123 -> Diode_SMD:D_MiniMELF
- D50: renamed from D9; footprint Diode_SMD:D_SOD-123 -> Diode_SMD:D_MiniMELF
- D51: renamed from D43; footprint Diode_SMD:D_SOD-123 -> Diode_SMD:D_MiniMELF
- D52: renamed from D60; footprint Diode_SMD:D_SOD-123 -> Diode_SMD:D_MiniMELF
- D53: renamed from D27; footprint Diode_SMD:D_SOD-123 -> Diode_SMD:D_MiniMELF
- D54: renamed from D81; footprint Diode_SMD:D_SOD-123 -> Diode_SMD:D_MiniMELF
- D55: renamed from D73; footprint Diode_SMD:D_SOD-123 -> Diode_SMD:D_MiniMELF
- D56: renamed from D44; footprint Diode_SMD:D_SOD-123 -> Diode_SMD:D_MiniMELF
- D57: renamed from D61; footprint Diode_SMD:D_SOD-123 -> Diode_SMD:D_MiniMELF
- D58: renamed from D10; footprint Diode_SMD:D_SOD-123 -> Diode_SMD:D_MiniMELF
- D59: renamed from D28; footprint Diode_SMD:D_SOD-123 -> Diode_SMD:D_MiniMELF
- D6: renamed from D64; footprint Diode_SMD:D_SOD-123 -> Diode_SMD:D_MiniMELF
- D60: renamed from D74; footprint Diode_SMD:D_SOD-123 -> Diode_SMD:D_MiniMELF
- D61: renamed from D82; footprint Diode_SMD:D_SOD-123 -> Diode_SMD:D_MiniMELF
- D62: renamed from D45; footprint Diode_SMD:D_SOD-123 -> Diode_SMD:D_MiniMELF
- D63: renamed from D62; footprint Diode_SMD:D_SOD-123 -> Diode_SMD:D_MiniMELF
- D64: renamed from D11; footprint Diode_SMD:D_SOD-123 -> Diode_SMD:D_MiniMELF
- D65: renamed from D29; footprint Diode_SMD:D_SOD-123 -> Diode_SMD:D_MiniMELF
- D66: renamed from D46; footprint Diode_SMD:D_SOD-123 -> Diode_SMD:D_MiniMELF
- D67: renamed from D83; footprint Diode_SMD:D_SOD-123 -> Diode_SMD:D_MiniMELF
- D68: renamed from D12; footprint Diode_SMD:D_SOD-123 -> Diode_SMD:D_MiniMELF
- D69: renamed from D75; footprint Diode_SMD:D_SOD-123 -> Diode_SMD:D_MiniMELF
- D7: renamed from D18; footprint Diode_SMD:D_SOD-123 -> Diode_SMD:D_MiniMELF
- D70: renamed from D63; footprint Diode_SMD:D_SOD-123 -> Diode_SMD:D_MiniMELF
- D71: renamed from D30; footprint Diode_SMD:D_SOD-123 -> Diode_SMD:D_MiniMELF
- D72: renamed from D47; footprint Diode_SMD:D_SOD-123 -> Diode_SMD:D_MiniMELF
- D73: renamed from D84; footprint Diode_SMD:D_SOD-123 -> Diode_SMD:D_MiniMELF
- D74: renamed from D13; footprint Diode_SMD:D_SOD-123 -> Diode_SMD:D_MiniMELF
- D75: renamed from D14; footprint Diode_SMD:D_SOD-123 -> Diode_SMD:D_MiniMELF
- D76: renamed from D31; footprint Diode_SMD:D_SOD-123 -> Diode_SMD:D_MiniMELF
- D77: renamed from D48; footprint Diode_SMD:D_SOD-123 -> Diode_SMD:D_MiniMELF
- D78: renamed from D85; footprint Diode_SMD:D_SOD-123 -> Diode_SMD:D_MiniMELF
- D79: renamed from D15; footprint Diode_SMD:D_SOD-123 -> Diode_SMD:D_MiniMELF
- D8: renamed from D78; footprint Diode_SMD:D_SOD-123 -> Diode_SMD:D_MiniMELF
- D80: renamed from D32; footprint Diode_SMD:D_SOD-123 -> Diode_SMD:D_MiniMELF
- D81: renamed from D49; footprint Diode_SMD:D_SOD-123 -> Diode_SMD:D_MiniMELF
- D82: renamed from D76; footprint Diode_SMD:D_SOD-123 -> Diode_SMD:D_MiniMELF
- D83: renamed from D86; footprint Diode_SMD:D_SOD-123 -> Diode_SMD:D_MiniMELF
- D84: renamed from D16; footprint Diode_SMD:D_SOD-123 -> Diode_SMD:D_MiniMELF
- D85: renamed from D33; footprint Diode_SMD:D_SOD-123 -> Diode_SMD:D_MiniMELF
- D86: renamed from D50; footprint Diode_SMD:D_SOD-123 -> Diode_SMD:D_MiniMELF
- D9: renamed from D35; footprint Diode_SMD:D_SOD-123 -> Diode_SMD:D_MiniMELF
- J1: value USB_B -> GCT USB4085; footprint Connector_USB:USB_C_Receptacle_Amphenol_12401548E4-2A_CircularHoles -> Connector_USB:USB_C_Receptacle_GCT_USB4085
- LED_0: renamed from LED_53; value MX_LED -> Led_Small
- LED_1: renamed from LED_7; value MX_LED -> Led_Small
- LED_2: renamed from LED_12; value MX_LED -> Led_Small
- LED_3: renamed from LED_18; value MX_LED -> Led_Small
- LED_4: renamed from LED_23; value MX_LED -> Led_Small
- LED_6: renamed from LED_32; value MX_LED -> Led_Small
- LED_7: renamed from LED_38; value MX_LED -> Led_Small
- LED_9: renamed from LED_48; value MX_LED -> Led_Small
- LED_A1: renamed from LED_10; value MX_LED -> Led_Small
- LED_B1: renamed from LED_33; value MX_LED -> Led_Small
- LED_BKSLSH1: renamed from LED_72; value MX_LED -> Led_Small
- LED_C1: renamed from LED_24; value MX_LED -> Led_Small
- LED_CAPS1: renamed from LED_5; value MX_LED -> Led_Small
- LED_COLON1: renamed from LED_57; value MX_LED -> Led_Small
- LED_COMMA1: renamed from LED_49; value MX_LED -> Led_Small
- LED_D1: renamed from LED_21; value MX_LED -> Led_Small
- LED_DEL1: renamed from LED_77; value MX_LED -> Led_Small
- LED_DOWN1: renamed from LED_83; value MX_LED -> Led_Small
- LED_E1: renamed from LED_20; value MX_LED -> Led_Small
- LED_END1: renamed from LED_81; value MX_LED -> Led_Small
- LED_ENTER1: renamed from LED_70; value MX_LED -> Led_Small
- LED_EQUAL1: renamed from LED_65; value MX_LED -> Led_Small
- LED_ESC1: renamed from LED_2; value Led_Small -> ESC
- LED_F0: renamed from LED_26; value MX_LED -> Led_Small
- LED_F1: renamed from LED_11; value MX_LED -> Led_Small
- LED_F11: renamed from LED_68; value MX_LED -> Led_Small
- LED_F12: renamed from LED_74; value MX_LED -> Led_Small
- LED_F2: renamed from LED_17; value MX_LED -> Led_Small
- LED_F3: renamed from LED_22; value MX_LED -> Led_Small
- LED_F4: renamed from LED_27; value MX_LED -> Led_Small
- LED_F6: renamed from LED_40; value MX_LED -> Led_Small
- LED_F7: renamed from LED_45; value MX_LED -> Led_Small
- LED_F9: renamed from LED_59; value MX_LED -> Led_Small
- LED_FN1: renamed from LED_61; value MX_LED -> Led_Small
- LED_FSLASH1: renamed from LED_60; value MX_LED -> Led_Small
- LED_G1: renamed from LED_31; value MX_LED -> Led_Small
- LED_H1: renamed from LED_37; value MX_LED -> Led_Small
- LED_I1: renamed from LED_46; value MX_LED -> Led_Small
- LED_J1: renamed from LED_42; value MX_LED -> Led_Small
- LED_K1: renamed from LED_47; value MX_LED -> Led_Small
- LED_L1: renamed from LED_52; value MX_LED -> Led_Small
- LED_LALT1: renamed from LED_15; value MX_LED -> Led_Small
- LED_LBRACE1: renamed from LED_62; value MX_LED -> Led_Small
- LED_LCTL1: renamed from LED_3; value MX_LED -> Led_Small
- LED_LEFT1: renamed from LED_78; value MX_LED -> Led_Small
- LED_LSHIFT1: renamed from LED_6; value MX_LED -> Led_Small
- LED_LSUP1: renamed from LED_8; value MX_LED -> Led_Small
- LED_M1: renamed from LED_44; value MX_LED -> Led_Small
- LED_N1: renamed from LED_39; value MX_LED -> Led_Small
- LED_O1: renamed from LED_51; value MX_LED -> Led_Small
- LED_P1: renamed from LED_56; value MX_LED -> Led_Small
- LED_PAUSE1: renamed from LED_84; value MX_LED -> Led_Small
- LED_PERIOD1: renamed from LED_55; value MX_LED -> Led_Small
- LED_PGDN1: renamed from LED_86; value MX_LED -> Led_Small
- LED_Q1: renamed from LED_9; value MX_LED -> Led_Small
- LED_QUOT1: renamed from LED_63; value MX_LED -> Led_Small
- LED_R1: renamed from LED_25; value MX_LED -> Led_Small
- LED_RALT1: renamed from LED_54; value MX_LED -> Led_Small
- LED_RBRACE1: renamed from LED_66; value MX_LED -> Led_Small
- LED_RCTL1: renamed from LED_73; value MX_LED -> Led_Small
- LED_RIGHT1: renamed from LED_87; value MX_LED -> Led_Small
- LED_RSHIFT1: renamed from LED_69; value MX_LED -> Led_Small
- LED_RSUP1: renamed from LED_67; value MX_LED -> Led_Small
- LED_S1: renamed from LED_16; value MX_LED -> Led_Small
- LED_SPACE1: renamed from LED_34; value MX_LED -> Led_Small
- LED_T1: renamed from LED_30; value MX_LED -> Led_Small
- LED_TAB1: renamed from LED_4; value MX_LED -> Led_Small
- LED_U1: renamed from LED_41; value MX_LED -> Led_Small
- LED_UNDSCR1: renamed from LED_58; value MX_LED -> Led_Small
- LED_UP1: renamed from LED_82; value MX_LED -> Led_Small
- LED_V1: renamed from LED_29; value MX_LED -> Led_Small
- LED_W1: renamed from LED_14; value MX_LED -> Led_Small
- LED_X1: renamed from LED_19; value MX_LED -> Led_Small
- LED_Y1: renamed from LED_36; value MX_LED -> Led_Small
- LED_Z1: renamed from LED_13; value MX_LED -> Led_Small
- Q1: footprint TO_SOT_Packages_SMD:SOT-23 -> Package_TO_SOT_SMD:SOT-23
- R77: value 330r -> 470
- SW_2: value MX_LED -> 2
- moved LED_DEL1 293.8 mm to (330.6, 71.7)
- moved LED_S1 283.2 mm to (92.3, 90.8)
- moved LED_LALT1 278.5 mm to (89.7, 128.5)
- moved LED_LEFT1 264.6 mm to (330.5, 128.7)
- moved R81 260.2 mm to (325.0, 29.3), turned to 90 degrees
- moved R80 255.1 mm to (300.3, 29.2), turned to 90 degrees
- moved LED_W1 246.9 mm to (87.6, 71.8)
- moved R82 238.9 mm to (324.8, 53.0), turned to 90 degrees
- moved LED_Z1 237.3 mm to (82.9, 109.7)
- moved R83 220.0 mm to (324.6, 72.0), turned to 90 degrees
- moved LED_B1 217.2 mm to (159.0, 109.7)
- moved R84 211.6 mm to (324.7, 128.9), turned to 90 degrees
- moved LED_2 210.3 mm to (78.0, 52.6)
- moved LED_6 195.5 mm to (154.1, 52.6)
- moved LED_EQUAL1 193.9 mm to (268.2, 52.6)
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- renumbered C1 to C4, C2 to C5, C3 to C6, R6 to R11, R7 to R12, R8 to R13, R9 to R14, R10 to R15, R11 to R16, R12 to R17, R13 to R18, R14 to R19, R92 to R2, R15 to R20, R16 to R21, R17 to R22, R18 to R23, R19 to R24, R20 to R25, R21 to R26, R22 to R27, R23 to R28, R24 to R29, R93 to R3, R25 to R30, R26 to R31, R27 to R32, R28 to R33, R30 to R35, R31 to R36, R32 to R37, R33 to R38, R34 to R39, R75 to R4, R35 to R40, R36 to R41, R37 to R42, R38 to R43, R39 to R44, R40 to R45, R41 to R46, R42 to R47, R43 to R48, R76 to R5, R45 to R50, R46 to R51, R47 to R52, R48 to R53, R49 to R54, R50 to R55, R51 to R56, R52 to R57, R53 to R58, R54 to R59, R1 to R6, R55 to R60, R56 to R61, R57 to R62, R58 to R63, R59 to R64, R60 to R65, R61 to R66, R62 to R67, R63 to R68, R64 to R69, R2 to R7, R65 to R70, R66 to R71, R67 to R72, R68 to R73, R69 to R74, R70 to R75, R71 to R76, R73 to R78, R74 to R79, R3 to R8, R78 to R80, R79 to R81, R80 to R82, R81 to R83, R82 to R84, R87 to R89, R4 to R9, R88 to R90, R89 to R91, R90 to R92, R91 to R93, SW_LBKT1 to SW_LBRACE1, SW_RBKT1 to SW_RBRACE1
Connections:
- J1 pad A4: VCC -> VBUS
- J1 pad A9: VCC -> VBUS
- J1 pad B4: VCC -> VBUS
- J1 pad B9: VCC -> VBUS
- LED_0 pad 1: (no net) -> BLGND
- LED_0 pad 2: (no net) -> Net-(LED_0-Pad2)
- LED_1 pad 1: (no net) -> BLGND
- LED_1 pad 2: (no net) -> Net-(LED_1-Pad2)
- LED_2 pad 1: (no net) -> BLGND
- LED_2 pad 2: (no net) -> Net-(LED_2-Pad2)
- LED_3 pad 1: (no net) -> BLGND
- LED_3 pad 2: (no net) -> Net-(LED_3-Pad2)
- LED_4 pad 1: (no net) -> BLGND
- LED_4 pad 2: (no net) -> Net-(LED_4-Pad2)
- LED_6 pad 1: (no net) -> BLGND
- LED_6 pad 2: (no net) -> Net-(LED_6-Pad2)
- LED_7 pad 1: (no net) -> BLGND
- LED_7 pad 2: (no net) -> Net-(LED_7-Pad2)
- LED_9 pad 1: (no net) -> BLGND
- LED_9 pad 2: (no net) -> Net-(LED_9-Pad2)
- LED_A1 pad 1: (no net) -> BLGND
- LED_A1 pad 2: (no net) -> Net-(LED_A1-Pad2)
- LED_B1 pad 1: (no net) -> BLGND
- LED_B1 pad 2: (no net) -> Net-(LED_B1-Pad2)
- LED_BKSLSH1 pad 1: (no net) -> BLGND
- LED_BKSLSH1 pad 2: (no net) -> Net-(LED_BKSLSH1-Pad2)
- LED_C1 pad 1: (no net) -> BLGND
- LED_C1 pad 2: (no net) -> Net-(LED_C1-Pad2)
- LED_CAPS1 pad 1: (no net) -> GND
- LED_CAPS1 pad 2: (no net) -> Net-(LED_CAPS1-Pad2)
- LED_COLON1 pad 1: (no net) -> BLGND
- LED_COLON1 pad 2: (no net) -> Net-(LED_COLON1-Pad2)
- LED_COMMA1 pad 1: (no net) -> BLGND
- LED_COMMA1 pad 2: (no net) -> Net-(LED_COMMA1-Pad2)
- LED_D1 pad 1: (no net) -> BLGND
- LED_D1 pad 2: (no net) -> Net-(LED_D1-Pad2)
- LED_DEL1 pad 1: (no net) -> BLGND
- LED_DEL1 pad 2: (no net) -> Net-(LED_DEL1-Pad2)
- LED_DOWN1 pad 1: (no net) -> BLGND
- LED_DOWN1 pad 2: (no net) -> Net-(LED_DOWN1-Pad2)
- LED_E1 pad 1: (no net) -> BLGND
- LED_E1 pad 2: (no net) -> Net-(LED_E1-Pad2)
- LED_END1 pad 1: (no net) -> BLGND
- LED_END1 pad 2: (no net) -> Net-(LED_END1-Pad2)
- LED_ENTER1 pad 1: (no net) -> BLGND
- LED_ENTER1 pad 2: (no net) -> Net-(LED_ENTER1-Pad2)
- LED_EQUAL1 pad 1: (no net) -> BLGND
- LED_EQUAL1 pad 2: (no net) -> Net-(LED_EQUAL1-Pad2)
- LED_ESC1 pad 1: (no net) -> BLGND
- LED_ESC1 pad 2: (no net) -> Net-(LED_ESC1-Pad2)
- LED_F0 pad 1: (no net) -> BLGND
- LED_F0 pad 2: (no net) -> Net-(LED_F0-Pad2)
- LED_F1 pad 1: (no net) -> BLGND
- LED_F1 pad 2: (no net) -> Net-(LED_F1-Pad2)
- LED_F11 pad 1: (no net) -> BLGND
- LED_F11 pad 2: (no net) -> Net-(LED_F11-Pad2)
- LED_F12 pad 1: (no net) -> BLGND
- LED_F12 pad 2: (no net) -> Net-(LED_F12-Pad2)
- LED_F2 pad 1: (no net) -> BLGND
- LED_F2 pad 2: (no net) -> Net-(LED_F2-Pad2)
- LED_F3 pad 1: (no net) -> BLGND
- LED_F3 pad 2: (no net) -> Net-(LED_F3-Pad2)
- LED_F4 pad 1: (no net) -> BLGND
- LED_F4 pad 2: (no net) -> Net-(LED_F4-Pad2)
- LED_F6 pad 1: (no net) -> BLGND
- LED_F6 pad 2: (no net) -> Net-(LED_F6-Pad2)
- LED_F7 pad 1: (no net) -> BLGND
- LED_F7 pad 2: (no net) -> Net-(LED_F7-Pad2)
- LED_F9 pad 1: (no net) -> BLGND
- LED_F9 pad 2: (no net) -> Net-(LED_F9-Pad2)
- LED_FN1 pad 1: (no net) -> GND
- LED_FN1 pad 2: (no net) -> Net-(LED_FN1-Pad2)
- LED_FSLASH1 pad 1: (no net) -> BLGND
- LED_FSLASH1 pad 2: (no net) -> Net-(LED_FSLASH1-Pad2)
- LED_G1 pad 1: (no net) -> BLGND
- LED_G1 pad 2: (no net) -> Net-(LED_G1-Pad2)
- LED_H1 pad 1: (no net) -> BLGND
- LED_H1 pad 2: (no net) -> Net-(LED_H1-Pad2)
- LED_I1 pad 1: (no net) -> BLGND
- LED_I1 pad 2: (no net) -> Net-(LED_I1-Pad2)
- LED_J1 pad 1: (no net) -> BLGND
- LED_J1 pad 2: (no net) -> Net-(LED_J1-Pad2)
- LED_K1 pad 1: (no net) -> BLGND
- LED_K1 pad 2: (no net) -> Net-(LED_K1-Pad2)
- LED_L1 pad 1: (no net) -> BLGND
- LED_L1 pad 2: (no net) -> Net-(LED_L1-Pad2)
- LED_LALT1 pad 1: (no net) -> BLGND
- LED_LALT1 pad 2: (no net) -> Net-(LED_LALT1-Pad2)
- LED_LBRACE1 pad 1: (no net) -> BLGND
- LED_LBRACE1 pad 2: (no net) -> Net-(LED_LBRACE1-Pad2)
- LED_LCTL1 pad 1: (no net) -> BLGND
- LED_LCTL1 pad 2: (no net) -> Net-(LED_LCTL1-Pad2)
- LED_LEFT1 pad 1: (no net) -> BLGND
- LED_LEFT1 pad 2: (no net) -> Net-(LED_LEFT1-Pad2)
- LED_LSHIFT1 pad 1: (no net) -> BLGND
- LED_LSHIFT1 pad 2: (no net) -> Net-(LED_LSHIFT1-Pad2)
- LED_LSUP1 pad 1: (no net) -> BLGND
- LED_LSUP1 pad 2: (no net) -> Net-(LED_LSUP1-Pad2)
- LED_M1 pad 1: (no net) -> BLGND
- LED_M1 pad 2: (no net) -> Net-(LED_M1-Pad2)
- LED_N1 pad 1: (no net) -> BLGND
- LED_N1 pad 2: (no net) -> Net-(LED_N1-Pad2)
- LED_O1 pad 1: (no net) -> BLGND
- LED_O1 pad 2: (no net) -> Net-(LED_O1-Pad2)
- LED_P1 pad 1: (no net) -> BLGND
- LED_P1 pad 2: (no net) -> Net-(LED_P1-Pad2)
- LED_PAUSE1 pad 1: (no net) -> BLGND
- LED_PAUSE1 pad 2: (no net) -> Net-(LED_PAUSE1-Pad2)
- LED_PERIOD1 pad 1: (no net) -> BLGND
- LED_PERIOD1 pad 2: (no net) -> Net-(LED_PERIOD1-Pad2)
- LED_PGDN1 pad 1: (no net) -> BLGND
- LED_PGDN1 pad 2: (no net) -> Net-(LED_PGDN1-Pad2)
- LED_Q1 pad 1: (no net) -> BLGND
- LED_Q1 pad 2: (no net) -> Net-(LED_Q1-Pad2)
- LED_QUOT1 pad 1: (no net) -> BLGND
- LED_QUOT1 pad 2: (no net) -> Net-(LED_QUOT1-Pad2)
- LED_R1 pad 1: (no net) -> BLGND
- LED_R1 pad 2: (no net) -> Net-(LED_R1-Pad2)
- LED_RALT1 pad 1: (no net) -> BLGND
- LED_RALT1 pad 2: (no net) -> Net-(LED_RALT1-Pad2)
- LED_RBRACE1 pad 1: (no net) -> BLGND
- LED_RBRACE1 pad 2: (no net) -> Net-(LED_RBRACE1-Pad2)
- LED_RCTL1 pad 1: (no net) -> BLGND
- LED_RCTL1 pad 2: (no net) -> Net-(LED_RCTL1-Pad2)
- LED_RIGHT1 pad 1: (no net) -> BLGND
- LED_RIGHT1 pad 2: (no net) -> Net-(LED_RIGHT1-Pad2)
- LED_RSHIFT1 pad 1: (no net) -> BLGND
- LED_RSHIFT1 pad 2: (no net) -> Net-(LED_RSHIFT1-Pad2)
- LED_RSUP1 pad 1: (no net) -> BLGND
- LED_RSUP1 pad 2: (no net) -> Net-(LED_RSUP1-Pad2)
- LED_S1 pad 1: (no net) -> BLGND
- LED_S1 pad 2: (no net) -> Net-(LED_S1-Pad2)
- LED_SPACE1 pad 1: (no net) -> BLGND
- LED_SPACE1 pad 2: (no net) -> Net-(LED_SPACE1-Pad2)
- LED_T1 pad 1: (no net) -> BLGND
- LED_T1 pad 2: (no net) -> Net-(LED_T1-Pad2)
- LED_TAB1 pad 1: (no net) -> BLGND
- LED_TAB1 pad 2: (no net) -> Net-(LED_TAB1-Pad2)
- LED_U1 pad 1: (no net) -> BLGND
- LED_U1 pad 2: (no net) -> Net-(LED_U1-Pad2)
- LED_UNDSCR1 pad 1: (no net) -> BLGND
- LED_UNDSCR1 pad 2: (no net) -> Net-(LED_UNDSCR1-Pad2)
- LED_UP1 pad 1: (no net) -> BLGND
- LED_UP1 pad 2: (no net) -> Net-(LED_UP1-Pad2)
- LED_V1 pad 1: (no net) -> BLGND
- LED_V1 pad 2: (no net) -> Net-(LED_V1-Pad2)
- LED_W1 pad 1: (no net) -> BLGND
- LED_W1 pad 2: (no net) -> Net-(LED_W1-Pad2)
- LED_X1 pad 1: (no net) -> BLGND
- LED_X1 pad 2: (no net) -> Net-(LED_X1-Pad2)
- LED_Y1 pad 1: (no net) -> BLGND
- LED_Y1 pad 2: (no net) -> Net-(LED_Y1-Pad2)
- LED_Z1 pad 1: (no net) -> BLGND
- LED_Z1 pad 2: (no net) -> Net-(LED_Z1-Pad2)
- Q1 pad 1: (no net) -> Net-(Q1-Pad1)
- Q1 pad 2: (no net) -> GND
- Q1 pad 3: (no net) -> BLGND
- R11 pad 1: (no net) -> Net-(LED_CAPS1-Pad2)
- R11 pad 2: (no net) -> CapsBL
- R12 pad 1: (no net) -> Net-(LED_LSHIFT1-Pad2)
- R12 pad 2: (no net) -> VCC
- R13 pad 1: (no net) -> Net-(LED_1-Pad2)
- R13 pad 2: (no net) -> VCC
- R14 pad 1: (no net) -> Net-(LED_LSUP1-Pad2)
- R14 pad 2: (no net) -> VCC
- R15 pad 1: (no net) -> Net-(LED_Q1-Pad2)
- R15 pad 2: (no net) -> VCC
- R16 pad 1: (no net) -> Net-(LED_A1-Pad2)
- R16 pad 2: (no net) -> VCC
- R17 pad 1: (no net) -> Net-(LED_F1-Pad2)
- R17 pad 2: (no net) -> VCC
- R18 pad 1: (no net) -> Net-(LED_2-Pad2)
- R18 pad 2: (no net) -> VCC
- R19 pad 1: (no net) -> Net-(LED_Z1-Pad2)
- R19 pad 2: (no net) -> VCC
- R20 pad 1: (no net) -> Net-(LED_W1-Pad2)
- R20 pad 2: (no net) -> VCC
- R21 pad 1: (no net) -> Net-(LED_LALT1-Pad2)
- R21 pad 2: (no net) -> VCC
- R22 pad 1: (no net) -> Net-(LED_S1-Pad2)
- R22 pad 2: (no net) -> VCC
- R23 pad 1: (no net) -> Net-(LED_F2-Pad2)
- R23 pad 2: (no net) -> VCC
- R24 pad 1: (no net) -> Net-(LED_3-Pad2)
- R24 pad 2: (no net) -> VCC
- R25 pad 1: (no net) -> Net-(LED_X1-Pad2)
- R25 pad 2: (no net) -> VCC
- R26 pad 1: (no net) -> Net-(LED_E1-Pad2)
- R26 pad 2: (no net) -> VCC
- R27 pad 1: (no net) -> Net-(LED_D1-Pad2)
- R27 pad 2: (no net) -> VCC
- R28 pad 1: (no net) -> Net-(LED_F3-Pad2)
- R28 pad 2: (no net) -> VCC
- R29 pad 1: (no net) -> Net-(LED_4-Pad2)
- R29 pad 2: (no net) -> VCC
- R30 pad 1: (no net) -> Net-(LED_C1-Pad2)
- R30 pad 2: (no net) -> VCC
- R31 pad 1: (no net) -> Net-(LED_R1-Pad2)
- R31 pad 2: (no net) -> VCC
- R32 pad 1: (no net) -> Net-(LED_F0-Pad2)
- R32 pad 2: (no net) -> VCC
- R33 pad 1: (no net) -> Net-(LED_F4-Pad2)
- R33 pad 2: (no net) -> VCC
- R35 pad 1: (no net) -> Net-(LED_V1-Pad2)
- R35 pad 2: (no net) -> VCC
- R36 pad 1: (no net) -> Net-(LED_T1-Pad2)
- R36 pad 2: (no net) -> VCC
- R37 pad 1: (no net) -> Net-(LED_G1-Pad2)
- R37 pad 2: (no net) -> VCC
- R38 pad 1: (no net) -> Net-(LED_6-Pad2)
- R38 pad 2: (no net) -> VCC
- R39 pad 1: (no net) -> Net-(LED_B1-Pad2)
- R39 pad 2: (no net) -> VCC
- R40 pad 1: (no net) -> Net-(LED_SPACE1-Pad2)
- R40 pad 2: (no net) -> VCC
- R41 pad 1: (no net) -> Net-(LED_F5-Pad2)
- R41 pad 2: (no net) -> VCC
- R42 pad 1: (no net) -> Net-(LED_Y1-Pad2)
- R42 pad 2: (no net) -> VCC
- R43 pad 1: (no net) -> Net-(LED_H1-Pad2)
- R43 pad 2: (no net) -> VCC
- R44 pad 1: (no net) -> Net-(LED_7-Pad2)
- R44 pad 2: (no net) -> VCC
- R45 pad 1: (no net) -> Net-(LED_N1-Pad2)
- R45 pad 2: (no net) -> VCC
- R46 pad 1: (no net) -> Net-(LED_F6-Pad2)
- R46 pad 2: (no net) -> VCC
- R47 pad 1: (no net) -> Net-(LED_U1-Pad2)
- R47 pad 2: (no net) -> VCC
- R48 pad 1: (no net) -> Net-(LED_J1-Pad2)
- R48 pad 2: (no net) -> VCC
- R50 pad 1: (no net) -> Net-(LED_M1-Pad2)
- R50 pad 2: (no net) -> VCC
- R51 pad 1: (no net) -> Net-(LED_F7-Pad2)
- R51 pad 2: (no net) -> VCC
- R52 pad 1: (no net) -> Net-(LED_I1-Pad2)
- R52 pad 2: (no net) -> VCC
- R53 pad 1: (no net) -> Net-(LED_K1-Pad2)
- R53 pad 2: (no net) -> VCC
- R54 pad 1: (no net) -> Net-(LED_9-Pad2)
- R54 pad 2: (no net) -> VCC
- R55 pad 1: (no net) -> Net-(LED_COMMA1-Pad2)
- R55 pad 2: (no net) -> VCC
- R56 pad 1: (no net) -> Net-(LED_F8-Pad2)
- R56 pad 2: (no net) -> VCC
- R57 pad 1: (no net) -> Net-(LED_O1-Pad2)
- R57 pad 2: (no net) -> VCC
- R58 pad 1: (no net) -> Net-(LED_L1-Pad2)
- R58 pad 2: (no net) -> VCC
- R59 pad 1: (no net) -> Net-(LED_0-Pad2)
- R59 pad 2: (no net) -> VCC
- R6 pad 1: (no net) -> Net-(LED_TILDE1-Pad2)
- R6 pad 2: (no net) -> VCC
- R60 pad 1: (no net) -> Net-(LED_RALT1-Pad2)
- R60 pad 2: (no net) -> VCC
- R61 pad 1: (no net) -> Net-(LED_PERIOD1-Pad2)
- R61 pad 2: (no net) -> VCC
- R62 pad 1: (no net) -> Net-(LED_P1-Pad2)
- R62 pad 2: (no net) -> VCC
- R63 pad 1: (no net) -> Net-(LED_COLON1-Pad2)
- R63 pad 2: (no net) -> VCC
- R64 pad 1: (no net) -> Net-(LED_UNDSCR1-Pad2)
- R64 pad 2: (no net) -> VCC
- R65 pad 1: (no net) -> Net-(LED_F9-Pad2)
- R65 pad 2: (no net) -> VCC
- R66 pad 1: (no net) -> Net-(LED_FSLASH1-Pad2)
- R66 pad 2: (no net) -> VCC
- R67 pad 1: (no net) -> Net-(LED_FN1-Pad2)
- R67 pad 2: (no net) -> FnBL
- R68 pad 1: (no net) -> Net-(LED_LBRACE1-Pad2)
- R68 pad 2: (no net) -> VCC
- R69 pad 1: (no net) -> Net-(LED_QUOT1-Pad2)
- R69 pad 2: (no net) -> VCC
- R7 pad 1: (no net) -> Net-(LED_ESC1-Pad2)
- R7 pad 2: (no net) -> VCC
- R70 pad 1: (no net) -> Net-(LED_F10-Pad2)
- R70 pad 2: (no net) -> VCC
- R71 pad 1: (no net) -> Net-(LED_EQUAL1-Pad2)
- R71 pad 2: (no net) -> VCC
- R72 pad 1: (no net) -> Net-(LED_RBRACE1-Pad2)
- R72 pad 2: (no net) -> VCC
- R73 pad 1: (no net) -> Net-(LED_RSUP1-Pad2)
- R73 pad 2: (no net) -> VCC
- R74 pad 1: (no net) -> Net-(LED_F11-Pad2)
- R74 pad 2: (no net) -> VCC
- R75 pad 1: (no net) -> Net-(LED_RSHIFT1-Pad2)
- R75 pad 2: (no net) -> VCC
- R76 pad 1: (no net) -> Net-(LED_ENTER1-Pad2)
- R76 pad 2: (no net) -> VCC
- R77 pad 1: VCC -> Net-(LED_BKSPC1-Pad2)
- R77 pad 2: GND -> VCC
- R78 pad 1: (no net) -> Net-(LED_BKSLSH1-Pad2)
- R78 pad 2: (no net) -> VCC
- R79 pad 1: (no net) -> Net-(LED_RCTL1-Pad2)
- R79 pad 2: (no net) -> VCC
- R8 pad 1: (no net) -> Net-(LED_LCTL1-Pad2)
- R8 pad 2: (no net) -> VCC
- R80 pad 1: (no net) -> Net-(LED_F12-Pad2)
- R80 pad 2: (no net) -> VCC
- R81 pad 1: (no net) -> Net-(LED_PRN1-Pad2)
- R81 pad 2: (no net) -> VCC
- R82 pad 1: (no net) -> Net-(LED_INS1-Pad2)
- R82 pad 2: (no net) -> VCC
- R83 pad 1: (no net) -> Net-(LED_DEL1-Pad2)
- R83 pad 2: (no net) -> VCC
- R84 pad 1: (no net) -> Net-(LED_LEFT1-Pad2)
- R84 pad 2: (no net) -> VCC
- R85 pad 1: (no net) -> Net-(LED_SCRL1-Pad2)
- R85 pad 2: (no net) -> ScrollBL
- R86 pad 1: (no net) -> Net-(LED_HOME1-Pad2)
- R86 pad 2: (no net) -> VCC
- R89 pad 1: (no net) -> Net-(LED_DOWN1-Pad2)
- R89 pad 2: (no net) -> VCC
- R9 pad 1: (no net) -> Net-(LED_TAB1-Pad2)
- R9 pad 2: (no net) -> VCC
- R90 pad 1: (no net) -> Net-(LED_PAUSE1-Pad2)
- R90 pad 2: (no net) -> VCC
- R91 pad 1: (no net) -> Net-(LED_PGUP1-Pad2)
- R91 pad 2: (no net) -> VCC
- R92 pad 1: (no net) -> Net-(LED_PGDN1-Pad2)
- R92 pad 2: (no net) -> VCC
- R93 pad 1: (no net) -> Net-(LED_RIGHT1-Pad2)
- R93 pad 2: (no net) -> VCC
Routing:
- net (no net): track 2484.7 -> 0.00 mm, vias 2 -> 0
- net GND: track 84.0 -> 513.7 mm, vias 9 -> 17
- net Net-(U1-Pad61): track 170.2 -> 0.02 mm, vias 2 -> 0
- net FnBL: track 142.3 -> 109.6 mm
- net Col8: track 299.9 -> 283.4 mm, vias 0 -> 1
- net Row6: track 380.3 -> 396.1 mm, vias 2 -> 4
- net VBUS: track 0.00 -> 15.8 mm
- net Row1: track 476.7 -> 463.6 mm
- net Col18: track 152.7 -> 165.3 mm, vias 5 -> 4
- net ScrollBL: track 80.7 -> 93.0 mm, vias 2 -> 4
- net Row5: track 338.6 -> 350.6 mm
- net /controller/XTAL1: track 16.9 -> 27.7 mm
- net /controller/MISO: track 7.96 -> 13.4 mm
- net Col2: track 399.1 -> 404.5 mm
- net Net-(D5-Pad2): track 0.00 -> 5.27 mm
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- added copper zone on F.Cu, net BLGND
- added copper zone on F.Cu, net GND
- removed copper zone on B.Cu, net GND
Other:
- board size 348.3 x 121 mm -> 348.1 x 120.9 mm
- net class Default: clearance 0.2 -> 0.15
- rule trace_clearance: 0.2 -> 0.15
- board text added: "ec0board v3 <3"
- board text removed: "ec0board v2"
