File: nummacro.kicad_pcb (KiCad board)
At the start: 2 copper layers, 348.1 x 120.9 mm, 370 parts, among them CON1 ISP, J1 GCT USB4085, Q1 Q_NPN_BEC, SW1 SW_RESET, SW2 SW_HWB, U1 AT90USB1286, Y1 16Mhz

Commit message: WIP USB-C 3d model, cleaned up main key matrix routing quite a bit
Parts:
- SW1, SW2: footprint Button_Switch_SMD:SW_SPST_B3SL-1002P -> Button_Switch_SMD:SW_SPST_EVQQ2
Routing:
- net /controller/XTAL1: track 27.7 -> 19.4 mm
- net GND: track 513.7 -> 520.5 mm, vias 17 -> 16
- net Col14: track 198.4 -> 194.7 mm
- net Col13: track 163.9 -> 160.2 mm
- net Col6: track 331.9 -> 334.5 mm
- net Col8: track 283.4 -> 286.0 mm
- net Col10: track 261.7 -> 264.2 mm
- net Col11: track 268.3 -> 270.9 mm
- net Col9: track 278.8 -> 281.3 mm
- net Col12: track 222.6 -> 225.1 mm
- net Col7: track 323.7 -> 326.2 mm
- net Col1: track 445.1 -> 443.5 mm
- net Col4: track 397.3 -> 395.9 mm
- net Col5: track 358.8 -> 357.5 mm
- net Col3: track 397.9 -> 396.6 mm
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
Commit message: Silkscreen overhaul to move everything to the back layer, moved diode symbols to silkscreen from fab layer. Regenerated gerbs.
Parts:
- moved D3 1.13 mm to (35.4, 138.5)
Routing:
- net GND: track 520.5 -> 517.8 mm
- net Net-(D3-Pad2): track 4.93 -> 3.35 mm
- net Row6: track 396.1 -> 395.4 mm
Other:
- outline, holes or cut-outs redrawn
- board text added: "USB-C 2.0"
- board text removed: "USB 2.0"

Commit message: v3 initial commit, USB-C, interactive BOM, rerouted and changed to use standard KiCad libs where possible
Parts:
- D1, D10, D11, D12, D13, D14, D15, D16, D17, D18, D19, D2, D20, D21, D22, D23, D24, D25, D26, D27, D28, D29, D3, D30, D31, D32, D33, D34, D35, D36, D37, D38, D39, D4, D40, D41, D42, D43, D44, D45, D46, D47, D48, D49, D5, D50, D51, D52, D53, D54, D55, D56, D57, D58, D59, D6, D60, D61, D62, D63, D64, D65, D66, D67, D68, D69, D7, D70, D71, D72, D73, D74, D75, D76, D77, D78, D79, D8, D80, D81, D82, D83, D84, D85, D86, D87, D9: value D -> LL4148
- LED_0, LED_1, LED_2, LED_3, LED_4, LED_5, LED_6, LED_7, LED_8, LED_9, LED_A1, LED_B1, LED_BKSLSH1, LED_BKSPC1, LED_C1, LED_CAPS1, LED_COLON1, LED_COMMA1, LED_D1, LED_DEL1, LED_DOWN1, LED_E1, LED_END1, LED_ENTER1, LED_EQUAL1, LED_F0, LED_F1, LED_F10, LED_F11, LED_F12, LED_F2, LED_F3, LED_F4, LED_F5, LED_F6, LED_F7, LED_F8, LED_F9, LED_FN1, LED_FSLASH1, LED_G1, LED_H1, LED_HOME1, LED_I1, LED_INS1, LED_J1, LED_K1, LED_L1, LED_LALT1, LED_LBRACE1, LED_LCTL1, LED_LEFT1, LED_LSHIFT1, LED_LSUP1, LED_M1, LED_N1, LED_O1, LED_P1, LED_PAUSE1, LED_PERIOD1, LED_PGDN1, LED_PGUP1, LED_PRN1, LED_Q1, LED_QUOT1, LED_R1, LED_RALT1, LED_RBRACE1, LED_RCTL1, LED_RIGHT1, LED_RSHIFT1, LED_RSUP1, LED_S1, LED_SCRL1, LED_SPACE1, LED_T1, LED_TAB1, LED_TILDE1, LED_U1, LED_UNDSCR1, LED_UP1, LED_V1, LED_W1, LED_X1, LED_Y1, LED_Z1: value Led_Small -> LED
- LED_ESC1: value ESC -> LED
- Q1: value Q_NPN_BEC -> MMBT3904
- SW1: value SW_RESET -> RESET
- SW2: value SW_HWB -> HWB
- SW_1: value MX_LED -> 1
- SW_10: value MX_LED -> 0
- SW_3: value MX_LED -> 3
- SW_4: value MX_LED -> 4
- SW_5: value MX_LED -> 5
- SW_6: value MX_LED -> 6
- SW_7: value MX_LED -> 7
- SW_8: value MX_LED -> 8
- SW_9: value MX_LED -> 9
- SW_A1: value MX_LED -> A
- SW_B1: value MX_LED -> B
- SW_BKSPC1: value MX_LED -> BKSPC
- SW_BSLSH1: value MX_LED -> BSLSH
- SW_C1: value MX_LED -> C
- SW_CAPS1: value MX_LED -> CAPS
- SW_COLON1: value MX_LED -> COLON
- SW_COMMA1: value MX_LED -> COMMA
- SW_D1: value MX_LED -> D
- SW_DEL1: value MX_LED -> DEL
- SW_DOWN1: value MX_LED -> DOWN
- SW_E1: value MX_LED -> E
- SW_END1: value MX_LED -> END
- SW_ENTER1: value MX_LED -> ENTER
- SW_EQUAL1: value MX_LED -> EQUAL
- SW_ESC1: value MX_LED -> ESC
- SW_F0: value MX_LED -> F
- SW_F1: value MX_LED -> F1
- SW_F10: value MX_LED -> F10
- SW_F11: value MX_LED -> F11
- SW_F12: value MX_LED -> F12
- SW_F2: value MX_LED -> F2
- SW_F3: value MX_LED -> F3
- SW_F4: value MX_LED -> F4
- SW_F5: value MX_LED -> F5
- SW_F6: value MX_LED -> F6
- SW_F7: value MX_LED -> F7
- SW_F8: value MX_LED -> F8
- SW_F9: value MX_LED -> F9
- SW_FSLASH1: value MX_LED -> FSLASH
- SW_FUNC1: value MX_LED -> FUNC
- SW_G1: value MX_LED -> G
- SW_H1: value MX_LED -> H
- SW_HOME1: value MX_LED -> HOME
- SW_I1: value MX_LED -> I
- SW_INS1: value MX_LED -> INS
- SW_J1: value MX_LED -> J
- SW_K1: value MX_LED -> K
- SW_L1: value MX_LED -> L
- SW_LALT1: value MX_LED -> LALT
- SW_LBRACE1: value MX_LED -> LBRACE
- SW_LCTRL1: value MX_LED -> LCTRL
- SW_LEFT1: value MX_LED -> LEFT
- SW_LSHIFT1: value MX_LED -> LSHIFT
- SW_LSUP1: value MX_LED -> LSUP
- SW_M1: value MX_LED -> M
- SW_N1: value MX_LED -> N
- SW_O1: value MX_LED -> O
- SW_P1: value MX_LED -> P
- SW_PAUSE1: value MX_LED -> PAUSE
- SW_PERIOD1: value MX_LED -> PERIOD
- SW_PGDN1: value MX_LED -> PGDN
- SW_PGUP1: value MX_LED -> PGUP
- SW_PRINT1: value MX_LED -> PRINT
- SW_Q1: value MX_LED -> Q
- SW_QUOT1: value MX_LED -> QUOT
- SW_R1: value MX_LED -> R
- SW_RALT1: value MX_LED -> RALT
- SW_RBRACE1: value MX_LED -> RBRACE
- SW_RCTL1: value MX_LED -> RCTL
- SW_RIGHT1: value MX_LED -> RIGHT
- SW_RSHIFT1: value MX_LED -> RSHIFT
- SW_RSUP1: value MX_LED -> RSUP
- SW_S1: value MX_LED -> S
- SW_SCROLL1: value MX_LED -> SCROLL
- SW_SPACE1: value MX_LED -> SPACE
- SW_T1: value MX_LED -> T
- SW_TAB1: value MX_LED -> TAB
- SW_TILDE1: value MX_LED -> TILDE
- SW_U1: value MX_LED -> U
- SW_UNDSCR1: value MX_LED -> UNDSCR
- SW_UP1: value MX_LED -> UP
- SW_V1: value MX_LED -> V
- SW_W1: value MX_LED -> W
- SW_X1: value MX_LED -> X
- SW_Y1: value MX_LED -> Y
- SW_Z1: value MX_LED -> Z
Connections:
- U1 pad 62: Net-(U1-Pad62) -> VCC
Routing:
- net VCC: track 10.1 -> 14.0 mm
