File: backlight.sch (KiCad schematic (older format))
At the start: 176 parts, among them Q1 Q_NPN_BEC

Commit message: v3 initial commit, USB-C, interactive BOM, rerouted and changed to use standard KiCad libs where possible
Parts:
- LED_0, LED_1, LED_2, LED_3, LED_4, LED_5, LED_6, LED_7, LED_8, LED_9, LED_A1, LED_B1, LED_BKSLSH1, LED_BKSPC1, LED_C1, LED_CAPS1, LED_COLON1, LED_COMMA1, LED_D1, LED_DEL1, LED_DOWN1, LED_E1, LED_END1, LED_ENTER1, LED_EQUAL1, LED_F0, LED_F1, LED_F10, LED_F11, LED_F12, LED_F2, LED_F3, LED_F4, LED_F5, LED_F6, LED_F7, LED_F8, LED_F9, LED_FN1, LED_FSLASH1, LED_G1, LED_H1, LED_HOME1, LED_I1, LED_INS1, LED_J1, LED_K1, LED_L1, LED_LALT1, LED_LBRACE1, LED_LCTL1, LED_LEFT1, LED_LSHIFT1, LED_LSUP1, LED_M1, LED_N1, LED_O1, LED_P1, LED_PAUSE1, LED_PERIOD1, LED_PGDN1, LED_PGUP1, LED_PRN1, LED_Q1, LED_QUOT1, LED_R1, LED_RALT1, LED_RBRACE1, LED_RCTL1, LED_RIGHT1, LED_RSHIFT1, LED_RSUP1, LED_S1, LED_SCRL1, LED_SPACE1, LED_T1, LED_TAB1, LED_TILDE1, LED_U1, LED_UNDSCR1, LED_UP1, LED_V1, LED_W1, LED_X1, LED_Y1, LED_Z1: value Led_Small -> LED; symbol device:LED -> Device:LED
- LED_ESC1: value ESC -> LED; symbol device:LED -> Device:LED
- Q1: value Q_NPN_BEC -> MMBT3904; symbol device:Q_NPN_BEC -> Transistor_BJT:MMBT3904
- R10: symbol device:R_Small -> Device:R_Small
- R11, R12, R13, R14, R15, R16, R17, R18, R19, R20, R21, R22, R23, R24, R25, R26, R27, R28, R29, R30, R31, R32, R33, R34, R35, R36, R37, R38, R39, R40, R41, R42, R43, R44, R45, R46, R47, R48, R49, R50, R51, R52, R53, R54, R55, R56, R57, R58, R59, R6, R60, R61, R62, R63, R64, R65, R66, R67, R68, R69, R7, R70, R71, R72, R73, R74, R75, R76, R77, R78, R79, R8, R80, R81, R82, R83, R84, R85, R86, R87, R88, R89, R9, R90, R91, R92, R93: symbol device:R -> Device:R
