File: controller.sch (KiCad schematic (older format))
At the start: 18 parts, among them CON1 ISP, J1 GCT USB4085, SW1 SW_RESET, SW2 SW_HWB, U1 AT90USB1286, Y1 16Mhz

Commit message: v3 initial commit, USB-C, interactive BOM, rerouted and changed to use standard KiCad libs where possible
Parts:
- C2, C3, C4, C5, C6, C7, C8: symbol device:C_Small -> Device:C_Small
- CON1: symbol nummacro-rescue:AVR-ISP-6-nummacro-rescue -> Connector:AVR-ISP-6
- D88: symbol device:D_Schottky -> nummacro-rescue:D_Schottky-device
- R2, R3, R4, R5: symbol device:R_Small -> Device:R_Small
- SW1: value SW_RESET -> RESET; symbol device:SW_PUSH -> Switch:SW_Push
- SW2: value SW_HWB -> HWB; symbol device:SW_PUSH -> Switch:SW_Push
- U1: symbol doragasu:AT90USB1286 -> MCU_Microchip_AVR:AT90USB1286-AU
- Y1: symbol device:Crystal_Small -> Device:Crystal_Small
Connections:
- net VCC: now also U1.62 (AREF)
- no-connect marks 19 -> 18
Other:
- moved on the sheet: C2, C3, C4, C5, C6, C7, C8, D88, R5, SW1, SW2, Y1
