File: keymatrix.sch (KiCad schematic (older format))
At the start: 174 parts

Commit message: v3 initial commit, USB-C, interactive BOM, rerouted and changed to use standard KiCad libs where possible
Parts:
- D1, D10, D11, D12, D13, D14, D15, D16, D17, D18, D19, D2, D20, D21, D22, D23, D24, D25, D26, D27, D28, D29, D3, D30, D31, D32, D33, D34, D35, D36, D37, D38, D39, D4, D40, D41, D42, D43, D44, D45, D46, D47, D48, D49, D5, D50, D51, D52, D53, D54, D55, D56, D57, D58, D59, D6, D60, D61, D62, D63, D64, D65, D66, D67, D68, D69, D7, D70, D71, D72, D73, D74, D75, D76, D77, D78, D79, D8, D80, D81, D82, D83, D84, D85, D86, D87, D9: value D -> LL4148; symbol device:D -> Diode:LL4148
- SW_1: value MX_LED -> 1
- SW_10: value MX_LED -> 0
- SW_3: value MX_LED -> 3
- SW_4: value MX_LED -> 4
- SW_5: value MX_LED -> 5
- SW_6: value MX_LED -> 6
- SW_7: value MX_LED -> 7
- SW_8: value MX_LED -> 8
- SW_9: value MX_LED -> 9
- SW_A1: value MX_LED -> A
- SW_B1: value MX_LED -> B
- SW_BKSPC1: value MX_LED -> BKSPC
- SW_BSLSH1: value MX_LED -> BSLSH
- SW_C1: value MX_LED -> C
- SW_CAPS1: value MX_LED -> CAPS
- SW_COLON1: value MX_LED -> COLON
- SW_COMMA1: value MX_LED -> COMMA
- SW_D1: value MX_LED -> D
- SW_DEL1: value MX_LED -> DEL
- SW_DOWN1: value MX_LED -> DOWN
- SW_E1: value MX_LED -> E
- SW_END1: value MX_LED -> END
- SW_ENTER1: value MX_LED -> ENTER
- SW_EQUAL1: value MX_LED -> EQUAL
- SW_ESC1: value MX_LED -> ESC
- SW_F0: value MX_LED -> F
- SW_F1: value MX_LED -> F1
- SW_F10: value MX_LED -> F10
- SW_F11: value MX_LED -> F11
- SW_F12: value MX_LED -> F12
- SW_F2: value MX_LED -> F2
- SW_F3: value MX_LED -> F3
- SW_F4: value MX_LED -> F4
- SW_F5: value MX_LED -> F5
- SW_F6: value MX_LED -> F6
- SW_F7: value MX_LED -> F7
- SW_F8: value MX_LED -> F8
- SW_F9: value MX_LED -> F9
- SW_FSLASH1: value MX_LED -> FSLASH
- SW_FUNC1: value MX_LED -> FUNC
- SW_G1: value MX_LED -> G
- SW_H1: value MX_LED -> H
- SW_HOME1: value MX_LED -> HOME
- SW_I1: value MX_LED -> I
- SW_INS1: value MX_LED -> INS
- SW_J1: value MX_LED -> J
- SW_K1: value MX_LED -> K
- SW_L1: value MX_LED -> L
- SW_LALT1: value MX_LED -> LALT
- SW_LBRACE1: value MX_LED -> LBRACE
- SW_LCTRL1: value MX_LED -> LCTRL
- SW_LEFT1: value MX_LED -> LEFT
- SW_LSHIFT1: value MX_LED -> LSHIFT
- SW_LSUP1: value MX_LED -> LSUP
- SW_M1: value MX_LED -> M
- SW_N1: value MX_LED -> N
- SW_O1: value MX_LED -> O
- SW_P1: value MX_LED -> P
- SW_PAUSE1: value MX_LED -> PAUSE
- SW_PERIOD1: value MX_LED -> PERIOD
- SW_PGDN1: value MX_LED -> PGDN
- SW_PGUP1: value MX_LED -> PGUP
- SW_PRINT1: value MX_LED -> PRINT
- SW_Q1: value MX_LED -> Q
- SW_QUOT1: value MX_LED -> QUOT
- SW_R1: value MX_LED -> R
- SW_RALT1: value MX_LED -> RALT
- SW_RBRACE1: value MX_LED -> RBRACE
- SW_RCTL1: value MX_LED -> RCTL
- SW_RIGHT1: value MX_LED -> RIGHT
- SW_RSHIFT1: value MX_LED -> RSHIFT
- SW_RSUP1: value MX_LED -> RSUP
- SW_S1: value MX_LED -> S
- SW_SCROLL1: value MX_LED -> SCROLL
- SW_SPACE1: value MX_LED -> SPACE
- SW_T1: value MX_LED -> T
- SW_TAB1: value MX_LED -> TAB
- SW_TILDE1: value MX_LED -> TILDE
- SW_U1: value MX_LED -> U
- SW_UNDSCR1: value MX_LED -> UNDSCR
- SW_UP1: value MX_LED -> UP
- SW_V1: value MX_LED -> V
- SW_W1: value MX_LED -> W
- SW_X1: value MX_LED -> X
- SW_Y1: value MX_LED -> Y
- SW_Z1: value MX_LED -> Z
